File: frontpanel/Toggle65.kicad_sch (KiCad schematic)
At the start: 117 parts, among them J1 Conn_01x02_Pin, J2 Conn_01x20_Pin, J4 Conn_01x20_Pin, SW10 On-None-Mom, SW11 RUN, SW13 Instruction/Cycle, SW14 RAM or Toggle, SW15 SP3T, SW16 SP3T, SW17 SP3T, SW18 SP3T, SW19 SP3T, SW2 SP3T, SW20 SP3T, SW21 SP3T, SW22 SP3T, SW23 Mom-Off-Mom, SW24 Mom-Off-Mom, SW25 Mom-Off-Mom, SW26 RAM or Toggle, SW27 RAM or Toggle, SW3 SP3T, SW4 SP3T, SW5 SP3T, SW6 SP3T, SW7 SP3T, SW8 SP3T, SW9 SP3T, U2 74HC74

Commit message: Minor improvements
Parts:
- added C6: 100nF, Capacitor_THT:C_Disc_D5.0mm_W2.5mm_P5.00mm, symbol Device:C_Small
Connections:
- net +5V: now also C6.1
- net GND: now also C6.2
Changed lines of the file:
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@@
 	)
 	(junction
+		(at 121.92 49.53)
+		(diameter 0)
+		(color 0 0 0 0)
+	)
+	(junction
+		(at 121.92 27.94)
+		(diameter 0)
+		(color 0 0 0 0)
+	)
+	(junction
 		(at 180.34 69.85)
 		(diameter 0)
@@
 	(wire
 		(pts
+			(xy 137.16 27.94) (xy 121.92 27.94)
+		)
+		(stroke
+			(width 0)
+			(type default)
+		)
+	)
+	(wire
+		(pts
 			(xy 147.32 118.11) (xy 156.21 118.11)
 		)
@@
 		)
 	)
+	(wire
+		(pts
+			(xy 137.16 43.18) (xy 137.16 49.53)
+		)
+		(stroke
+			(width 0)
+			(type default)
+		)
+	)
 	(bus
 		(pts
@@
 	(wire
 		(pts
+			(xy 121.92 27.94) (xy 121.92 29.21)
+		)
+		(stroke
+			(width 0)
+			(type default)
+		)
+	)
+	(wire
+		(pts
 			(xy 128.27 135.89) (xy 134.62 135.89)
 		)
@@
 	(wire
 		(pts
+			(xy 137.16 38.1) (xy 137.16 27.94)
+		)
+		(stroke
+			(width 0)
+			(type default)
+		)
+	)
+	(wire
+		(pts
 			(xy 67.31 93.98) (xy 72.39 93.98)
 		)
@@
 	(wire
 		(pts
-			(xy 121.92 26.67) (xy 121.92 29.21)
+			(xy 121.92 26.67) (xy 121.92 27.94)
 		)
 		(stroke
@@
 	(wire
 		(pts
+			(xy 137.16 49.53) (xy 121.92 49.53)
+		)
+		(stroke
+			(width 0)
+			(type default)
+		)
+	)
+	(wire
+		(pts
 			(xy 90.17 93.98) (xy 90.17 96.52)
 		)
@@
 					(unit 1)
 				)
+			)
+		)
+	)
+	(symbol
+		(lib_id "Device:C_Small")
+		(at 137.16 40.64 0)
+		(unit 1)
+		(body_style 1)
+		(exclude_from_sim no)
+		(in_bom yes)
+		(on_board yes)
+		(in_pos_files yes)
+		(dnp no)
+		(fields_autoplaced yes)
+		(property "Reference" "C6"
+			(at 139.7 39.3762 0)
+			(show_name no)
+			(do_not_autoplace no)
+			(effects
+				(font
+					(size 1.27 1.27)
+				)
+				(justify left)
+			)
+		)
+		(property "Value" "100nF"
+			(at 139.7 41.9162 0)
+			(show_name no)
+			(do_not_autoplace no)
+			(effects
+				(font
+					(size 1.27 1.27)
+				)
+				(justify left)
+			)
+		)
+		(property "Footprint" "Capacitor_THT:C_Disc_D5.0mm_W2.5mm_P5.00mm"
+			(at 137.16 40.64 0)
+			(hide yes)
+			(show_name no)
+			(do_not_autoplace no)
+			(effects
+				(font
+					(size 1.27 1.27)
+				)
+			)
+		)
+		(property "Datasheet" ""
+			(at 137.16 40.64 0)
+			(hide yes)
+			(show_name no)
+			(do_not_autoplace no)
+			(effects
+				(font
+					(size 1.27 1.27)
+				)
+			)
+		)
+		(property "Description" ""
+			(at 137.16 40.64 0)
+			(show_name no)
+			(do_not_autoplace no)
+			(effects
+				(font
+					(size 1.27 1.27)
+				)
+			)
+		)
+		(property "LCSC" "C49678"
+			(at 137.16 40.64 0)
+			(hide yes)
+			(show_name no)
+			(do_not_autoplace no)
+			(effects
+				(font
+					(size 1.27 1.27)
+				)
+			)
+		)
+		(pin "1"
+		)
+		(pin "2"
+		)
+		(instances
+			(project "Toggle65"
+				(path "/952348e6-14ff-4dd8-97a2-6ef53ae7757e"
+					(reference "C6")
+					(unit 1)
+				)

Commit message: Motherboard finished
Parts:
- added H1, H2, H3, H4: MountingHole, MountingHole:MountingHole_3.2mm_M3_DIN965, symbol Mechanical:MountingHole
