File: frontpanel/Toggle65.kicad_pcb (KiCad board)
At the start: 2 copper layers, 144.8 x 94 mm, 121 parts, among them J1 Conn_01x02_Pin, J2 Conn_01x20_Pin, J4 Conn_01x20_Pin, SW10 On-None-Mom, SW11 RUN, SW13 Instruction/Cycle, SW14 RAM or Toggle, SW15 SP3T, SW16 SP3T, SW17 SP3T, SW18 SP3T, SW19 SP3T, SW2 SP3T, SW20 SP3T, SW21 SP3T, SW22 SP3T, SW23 Mom-Off-Mom, SW24 Mom-Off-Mom, SW25 Mom-Off-Mom, SW26 RAM or Toggle, SW27 RAM or Toggle, SW3 SP3T, SW4 SP3T, SW5 SP3T, SW6 SP3T, SW7 SP3T, SW8 SP3T, SW9 SP3T, U2 74HC74

Commit message: Minor improvements
Parts:
- added C6: 100nF, Capacitor_THT:C_Disc_D5.0mm_W2.5mm_P5.00mm, F.Cu at (138.4, 64.2)
Routing:
- net +5V: track 432.0 -> 434.6 mm
- net RDY: track 74.7 -> 76.0 mm
- net LDMSBA: track 197.6 -> 198.7 mm
- net SYNC: track 86.7 -> 87.6 mm

Commit message: Motherboard finished
Parts:
- moved D5 0.22 mm to (126.5, 25.8)
- moved D1 0.20 mm to (162.0, 25.8)
- moved D12 0.20 mm to (61.7, 25.8)
- moved D13 0.20 mm to (52.8, 25.8)
- moved D14 0.20 mm to (43.9, 25.8)
- moved D16 0.20 mm to (26.1, 25.8)
- moved D11 0.20 mm to (70.6, 25.8)
- moved D15 0.20 mm to (35.0, 25.8)
- moved D6 0.20 mm to (117.6, 25.8)
- moved D7 0.20 mm to (108.7, 25.8)
- moved D8 0.20 mm to (99.8, 25.8)
- moved D2 0.19 mm to (153.1, 25.8)
- moved D9 0.19 mm to (88.3, 25.8)
- moved D10 0.19 mm to (79.4, 25.8)
- moved D3 0.19 mm to (144.2, 25.8)
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Other:
- board text added: "Power"
- board text removed: "System"

Commit message: Cleanup
Parts:
- moved R56 5.59 mm to (92.8, 84.5), turned to 0 degrees
- moved R15 2.92 mm to (44.5, 42.2)
- moved SW26 0.68 mm to (121.9, 65.0)
- moved R68 0.51 mm to (97.9, 91.4), turned to 180 degrees
- moved SW27 0.25 mm to (50.8, 65.0)
Routing:
- net +5V: track 434.6 -> 456.4 mm, vias 8 -> 4
- net GND: track 82.8 -> 61.5 mm
- net ~{WE}OVR: track 74.6 -> 82.1 mm, vias 2 -> 0
- net B15: track 78.9 -> 84.7 mm
- net ~{RST}: track 64.2 -> 58.8 mm, vias 2 -> 0
- net B3: track 64.4 -> 61.1 mm
- net ~{OE}OVR: track 63.3 -> 66.3 mm
- net B5: track 92.7 -> 90.1 mm
- net Net-(D17-K): track 10.0 -> 7.51 mm
- net B8: track 140.3 -> 138.0 mm
- net B9: track 130.1 -> 128.1 mm
- net B14: track 81.0 -> 82.9 mm
- net B10: track 120.4 -> 118.5 mm
- net Net-(U2A-D): track 96.6 -> 95.0 mm
- net Net-(D36-K): track 4.98 -> 6.54 mm
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Other:
- board text added: "6502 Microcomputer"
- board text added: "Address Bus"
- board text added: "Clock"
- board text added: "Toggle65"
