File: motherboard/motherboard.kicad_pcb (KiCad board)
At the start: 2 copper layers, 144.8 x 94 mm, 37 parts, among them J1 Conn_01x20_Pin, J3 Conn_01x20_Pin, J4 USB2.0_16P, U1 74LS573, U3 74HC132, U4 74HC245, U5 74HC245, U6 HM62256BLP, U7 R6507, U8 NE555P, U9 74HC132

Commit message: Minor improvements
Parts:
- moved D2 2.44 mm to (82.5, 67.0)
- moved D1 2.06 mm to (82.5, 63.5)
- moved U7 0.52 mm to (168.9, 31.0)
Routing:
- net VBAT: track 29.1 -> 32.4 mm
- net +5V: track 498.9 -> 501.7 mm
- net GND: track 199.9 -> 198.5 mm
- net Ø1: track 127.7 -> 126.7 mm
- net B11: track 172.6 -> 173.5 mm
- net Net-(D1-K): track 158.1 -> 157.2 mm
- net ~{WE}OVR: track 73.1 -> 72.3 mm
- net A10: track 12.0 -> 11.2 mm
- net A5: track 67.6 -> 67.0 mm
- net A4: track 65.0 -> 64.4 mm
- net D3: track 194.4 -> 195.0 mm
- net D4: track 185.3 -> 185.8 mm
- net Net-(U7-R/~{W}): track 38.5 -> 39.0 mm
- net A12: track 24.7 -> 25.2 mm
- net A11: track 18.1 -> 17.6 mm
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
Commit message: Motherboard finished
Parts:
- added R43: 4k7, Resistor_THT:R_Axial_DIN0204_L3.6mm_D1.6mm_P5.08mm_Horizontal, F.Cu at (127.6, 48.3)
- added R44: 4k7, Resistor_THT:R_Axial_DIN0204_L3.6mm_D1.6mm_P5.08mm_Horizontal, F.Cu at (124.4, 48.3)
- added R45: 4k7, Resistor_THT:R_Axial_DIN0204_L3.6mm_D1.6mm_P5.08mm_Horizontal, F.Cu at (121.3, 48.3)
Routing:
- net A15: track 0.00 -> 4.07 mm
- net A13: track 0.00 -> 4.05 mm
- net A14: track 0.00 -> 3.82 mm
- net VBAT: track 32.4 -> 31.1 mm
- net D7: track 155.7 -> 156.6 mm
- net B11: track 173.5 -> 172.7 mm

Commit message: Cleanup
Parts:
- added R46: 4k7, Resistor_THT:R_Axial_DIN0204_L3.6mm_D1.6mm_P5.08mm_Horizontal, F.Cu at (181.6, 92.5)
Connections:
- U3 pad 4: Net-(U7-R/~{W}) -> Ø0
- U3 pad 5: Net-(U7-R/~{W}) -> Ø0
- U7 pad 26: Net-(U7-R/~{W}) -> Ø0
Routing:
- net Net-(U7-R/~{W}): track 39.0 -> 0.00 mm, vias 2 -> 0
- net Ø0: track 119.7 -> 158.7 mm, vias 4 -> 6
- net ~{WE}OVR: track 72.3 -> 74.5 mm
- net GND: track 198.5 -> 200.5 mm
Changed lines of the file:
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@@
 	(footprint "Resistor_THT:R_Axial_DIN0204_L3.6mm_D1.6mm_P5.08mm_Horizontal"
 		(layer "F.Cu")
+		(at 181.5592 92.5068 90)
+		(descr "Resistor, Axial_DIN0204 series, Axial, Horizontal, pin pitch=5.08mm, 0.167W, length*diameter=3.6*1.6mm^2, http://cdn-reichelt.de/documents/datenblatt/B400/1_4W%23YAG.pdf")
+		(tags "Resistor Axial_DIN0204 series Axial Horizontal pin pitch 5.08mm 0.167W length 3.6mm diameter 1.6mm")
+		(property "Reference" "R46"
+			(at 2.54 -1.92 90)
+			(layer "F.SilkS")
+			(effects
+				(font
+					(size 1 1)
+					(thickness 0.15)
+				)
+			)
+		)
+		(property "Value" "4k7"
+			(at 2.54 1.92 90)
+			(layer "F.Fab")
+			(effects
+				(font
+					(size 1 1)
+					(thickness 0.15)
+				)
+			)
+		)
+		(property "Datasheet" ""
+			(at 0 0 90)
+			(layer "F.Fab")
+			(hide yes)
+			(effects
+				(font
+					(size 1.27 1.27)
+				)
+			)
+		)
+		(property "Description" ""
+			(at 0 0 90)
+			(layer "F.Fab")
+			(hide yes)
+			(effects
+				(font
+					(size 1.27 1.27)
+				)
+			)
+		)
+		(property "KiLib_Generator" "resistor/THT"
+			(at 0 0 90)
+			(layer "F.SilkS")
+			(hide yes)
+			(effects
+				(font
+					(size 1 1)
+					(thickness 0.15)
+				)
+			)
+		)
+		(property ki_fp_filters "R_*")
+		(sheetname "/")
+		(sheetfile "motherboard.kicad_sch")
+		(units
+			(unit
+				(name "A")
+				(pins "1" "2")
+			)
+		)
+		(attr through_hole)
+		(duplicate_pad_numbers_are_jumpers no)
+		(fp_line
+			(start 0.62 -0.92)
+			(end 4.46 -0.92)
+			(stroke
+				(width 0.12)
+				(type solid)
+			)
+			(layer "F.SilkS")
+		)
+		(fp_line
+			(start 0.62 0.92)
+			(end 4.46 0.92)
+			(stroke
+				(width 0.12)
+				(type solid)
+			)
+			(layer "F.SilkS")
+		)
+		(fp_poly
+			(pts
+				(xy -0.95 -1.050001) (xy 6.03 -1.05) (xy 6.03 1.05) (xy -0.95 1.050001)
+			)
+			(stroke
+				(width 0.05)
+				(type solid)
+			)
+			(fill no)
+			(layer "F.CrtYd")
+		)
+		(fp_line
+			(start 5.079999 0)
+			(end 4.339999 0)
+			(stroke
+				(width 0.1)
+				(type solid)
+			)
+			(layer "F.Fab")
+		)
+		(fp_line
+			(start 0 0)
+			(end 0.74 0)
+			(stroke
+				(width 0.1)
+				(type solid)
+			)
+			(layer "F.Fab")
+		)
+		(fp_poly
+			(pts
+				(xy 0.74 -0.799999) (xy 4.34 -0.8) (xy 4.34 0.8) (xy 0.74 0.799999)
+			)
+			(stroke
+				(width 0.1)
+				(type solid)
+			)
+			(fill no)
+			(layer "F.Fab")
+		)
+		(fp_text user "${REFERENCE}"
+			(at 2.54 0 90)
+			(layer "F.Fab")
+			(effects
+				(font
+					(size 0.72 0.72)
+					(thickness 0.108)
+				)
+			)
+		)
+		(pad "1" thru_hole circle
+			(at 0 0 90)
+			(size 1.4 1.4)
+			(drill 0.7)
+			(layers "*.Cu" "*.Mask")
+			(remove_unused_layers no)
+			(net "GND")
+			(pintype "passive")
+		)
+		(pad "2" thru_hole circle
+			(at 5.079999 0 90)
+			(size 1.4 1.4)
+			(drill 0.7)
+			(layers "*.Cu" "*.Mask")
+			(remove_unused_layers no)
+			(net "~{WE}OVR")
+			(pintype "passive")
+		)
+		(embedded_fonts no)
+		(model "${KICAD10_3DMODEL_DIR}/Resistor_THT.3dshapes/R_Axial_DIN0204_L3.6mm_D1.6mm_P5.08mm_Horizontal.step"
+			(offset
+				(xyz 0 0 0)
+			)
+			(scale
+				(xyz 1 1 1)
+			)
+			(rotate
+				(xyz 0 0 0)
+			)
+		)
+	)
+	(footprint "Resistor_THT:R_Axial_DIN0204_L3.6mm_D1.6mm_P5.08mm_Horizontal"
+		(layer "F.Cu")
 		(at 127.585 48.26 -90)
 		(descr "Resistor, Axial_DIN0204 series, Axial, Horizontal, pin pitch=5.08mm, 0.167W, length*diameter=3.6*1.6mm^2, http://cdn-reichelt.de/documents/datenblatt/B400/1_4W%23YAG.pdf")
@@
 			(layers "*.Cu" "*.Mask")
 			(remove_unused_layers no)
-			(net "Net-(U7-R{slash}~{W})")
+			(net "Ø0")
 			(pintype "input")
 		)
@@
 			(layers "*.Cu" "*.Mask")
 			(remove_unused_layers no)
-			(net "Net-(U7-R{slash}~{W})")
+			(net "Ø0")
 			(pintype "input")
 		)
@@
 			(layers "*.Cu" "*.Mask")
 			(remove_unused_layers no)
-			(net "Net-(U7-R{slash}~{W})")
+			(net "Ø0")
 			(pinfunction "R/~{W}_26")
 			(pintype "output")
@@
 	)
 	(segment
+		(start 180.5178 92.5068)
+		(end 179.832 91.821)
+		(width 0.4)
+		(layer "B.Cu")
+		(net "GND")
+	)
+	(segment
 		(start 117.856 74.295)
 		(end 118.745 74.295)
@@
 	)
 	(segment
+		(start 181.5592 92.5068)
+		(end 180.5178 92.5068)
+		(width 0.4)
+		(layer "B.Cu")
+		(net "GND")
+	)
+	(segment
 		(start 127.635 75.897503)
 		(end 126.032497 74.295)
@@
 	)
 	(segment
+		(start 127.585 53.339999)
+		(end 127.585 56.565)
+		(width 0.4)
+		(layer "B.Cu")
+		(net "A13")
+	)
+	(segment
+		(start 127.585 56.565)
+		(end 127 57.15)
+		(width 0.4)
+		(layer "B.Cu")
+		(net "A13")
+	)
+	(segment
 		(start 169.186421 92.917107)
 		(end 168.737973 92.917107)
@@
 	)
 	(segment
+		(start 180.543199 87.426801)
+		(end 179.705 88.265)
+		(width 0.4)
+		(layer "B.Cu")
+		(net "~{WE}OVR")
+	)
+	(segment
 		(start 128.27 81.285)
 		(end 128.27 83.82)
@@
 	)
 	(segment
+		(start 181.5592 87.426801)
+		(end 180.543199 87.426801)
+		(width 0.4)
+		(layer "B.Cu")
+		(net "~{WE}OVR")
+	)
+	(segment
 		(start 176.543264 88.939314)
 		(end 176.94695 89.343)
@@
 	)
 	(segment
+		(start 171.45 41.91)
+		(end 188.214 50.546)
+		(width 0.5)
+		(layer "F.Cu")
+		(net "Ø0")
+	)
+	(segment
 		(start 166.738 86.5)
 		(end 137.3 86.5)
@@
 	)
 	(via
+		(at 171.45 41.91)
+		(size 1.2)
+		(drill 0.8)
+		(layers "F.Cu" "B.Cu")
+		(net "Ø0")
+	)
+	(via
 		(at 136.942299 86.142299)
 		(size 1.2)
@@
 	)
 	(via
+		(at 188.214 50.546)
+		(size 1.2)
+		(drill 0.8)
+		(layers "F.Cu" "B.Cu")
+		(net "Ø0")
+	)
+	(via
 		(at 191.643 54.737)
 		(size 1.2)
@@
 	)
 	(segment
+		(start 163.83 46.24)
+		(end 163.83 43.815)
+		(width 0.5)
+		(layer "B.Cu")
+		(net "Ø0")
+	)
+	(segment
+		(start 186.73 57.15)
+		(end 184.19 57.15)
+		(width 0.5)
+		(layer "B.Cu")
+		(net "Ø0")
+	)
+	(segment
 		(start 191.81 57.15)
 		(end 194.35 57.15)
@@
 	)
 	(segment
+		(start 163.83 43.815)
+		(end 165.735 41.91)
+		(width 0.5)
+		(layer "B.Cu")
+		(net "Ø0")
+	)
+	(segment
+		(start 165.735 41.91)
+		(end 171.45 41.91)
+		(width 0.5)
+		(layer "B.Cu")
+		(net "Ø0")
+	)
+	(segment
 		(start 191.81 60.285)
 		(end 191.81 57.15)
@@
 	)
 	(segment
-		(start 171.45 41.91)
-		(end 188.214 50.546)
-		(width 0.5)
-		(layer "F.Cu")
-		(net "Net-(U7-R{slash}~{W})")
-	)
-	(via
-		(at 171.45 41.91)
-		(size 1.2)
-		(drill 0.8)
-		(layers "F.Cu" "B.Cu")
-		(net "Net-(U7-R{slash}~{W})")
-	)
-	(via
-		(at 188.214 50.546)
-		(size 1.2)
-		(drill 0.8)
-		(layers "F.Cu" "B.Cu")
-		(net "Net-(U7-R{slash}~{W})")
-	)
-	(segment
-		(start 163.83 46.24)
-		(end 163.83 43.815)
-		(width 0.5)
-		(layer "B.Cu")
-		(net "Net-(U7-R{slash}~{W})")
-	)
-	(segment
-		(start 186.73 57.15)
-		(end 184.19 57.15)
-		(width 0.5)
-		(layer "B.Cu")
-		(net "Net-(U7-R{slash}~{W})")
-	)
-	(segment
-		(start 163.83 43.815)
-		(end 165.735 41.91)
-		(width 0.5)
-		(layer "B.Cu")
-		(net "Net-(U7-R{slash}~{W})")
-	)
-	(segment
-		(start 165.735 41.91)
-		(end 171.45 41.91)
-		(width 0.5)
-		(layer "B.Cu")
-		(net "Net-(U7-R{slash}~{W})")
-	)
-	(segment
 		(start 186.73 57.15)
 		(end 188.214 50.546)
 		(width 0.5)
 		(layer "B.Cu")
-		(net "Net-(U7-R{slash}~{W})")
+		(net "Ø0")
 	)
 	(segment
@@
 	)
 	(segment
-		(start 127.585 53.339999)
-		(end 127.585 56.565)
-		(width 0.4)
-		(layer "B.Cu")
-		(net "A13")
-	)
-	(segment
-		(start 127.585 56.565)
-		(end 127 57.15)
-		(width 0.4)
-		(layer "B.Cu")
-		(net "A13")
-	)
-	(segment
