File: motherboard/motherboard.kicad_sch (KiCad schematic)
At the start: 37 parts, among them J1 Conn_01x20_Pin, J3 Conn_01x20_Pin, J4 USB2.0_16P, U1 74LS573, U3 74HC132, U4 74HC245, U5 74HC245, U6 HM62256BLP, U7 R6507, U8 NE555P, U9 74HC132

Commit message: Motherboard finished
Parts:
- added R43, R44, R45: 4k7, Resistor_THT:R_Axial_DIN0204_L3.6mm_D1.6mm_P5.08mm_Horizontal, symbol Device:R_Small
Connections:
- net A13: now also R43.2
- net A14: now also R44.2
- net A15: now also R45.2
- net GND: now also R43.1, R44.1, R45.1

Commit message: Cleanup
Parts:
- added R46: 4k7, Resistor_THT:R_Axial_DIN0204_L3.6mm_D1.6mm_P5.08mm_Horizontal, symbol Device:R_Small
- C1: now not fitted
Connections:
- net GND: now also R46.1
- net ~{WE}OVR: now also R46.2
- net Ø0: now also U3.4, U3.5, U7.26 (R/~{W})
Other:
- moved on the sheet: U9A, U9B
Changed lines of the file:
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@@
 	)
 	(junction
+		(at 173.99 161.29)
+		(diameter 0)
+		(color 0 0 0 0)
+	)
+	(junction
 		(at 148.59 138.43)
 		(diameter 0)
@@
 	)
 	(junction
+		(at 142.24 156.21)
+		(diameter 0)
+		(color 0 0 0 0)
+	)
+	(junction
 		(at 144.78 46.99)
 		(diameter 0)
@@
 	)
 	(junction
-		(at 143.51 156.21)
-		(diameter 0)
-		(color 0 0 0 0)
-	)
-	(junction
 		(at 53.34 130.81)
 		(diameter 0)
@@
 	(wire
 		(pts
-			(xy 128.27 147.32) (xy 135.89 147.32)
+			(xy 127 147.32) (xy 135.89 147.32)
 		)
 		(stroke
@@
 	(wire
 		(pts
-			(xy 143.51 153.67) (xy 143.51 156.21)
+			(xy 142.24 153.67) (xy 142.24 156.21)
 		)
 		(stroke
@@
 	(wire
 		(pts
-			(xy 128.27 156.21) (xy 128.27 147.32)
+			(xy 127 156.21) (xy 127 147.32)
 		)
 		(stroke
@@
 		)
 	)
+	(wire
+		(pts
+			(xy 166.37 153.67) (xy 158.75 153.67)
+		)
+		(stroke
+			(width 0)
+			(type default)
+		)
+	)
 	(bus
 		(pts
@@
 	(wire
 		(pts
+			(xy 173.99 161.29) (xy 173.99 165.1)
+		)
+		(stroke
+			(width 0)
+			(type default)
+		)
+	)
+	(wire
+		(pts
 			(xy 189.23 110.49) (xy 190.5 110.49)
 		)
@@
 	(wire
 		(pts
-			(xy 143.51 156.21) (xy 143.51 158.75)
+			(xy 142.24 156.21) (xy 142.24 158.75)
 		)
 		(stroke
@@
 	(wire
 		(pts
-			(xy 187.96 139.7) (xy 226.06 139.7)
+			(xy 187.96 140.97) (xy 215.9 140.97)
 		)
 		(stroke
@@
 	(wire
 		(pts
-			(xy 187.96 156.21) (xy 195.58 156.21)
+			(xy 173.99 156.21) (xy 195.58 156.21)
 		)
 		(stroke
@@
 	(wire
 		(pts
-			(xy 187.96 140.97) (xy 187.96 139.7)
-		)
-		(stroke
-			(width 0)
-			(type default)
-		)
-	)
-	(wire
-		(pts
 			(xy 135.89 120.65) (xy 143.51 120.65)
 		)
@@
 		)
 	)
+	(wire
+		(pts
+			(xy 142.24 156.21) (xy 143.51 156.21)
+		)
+		(stroke
+			(width 0)
+			(type default)
+		)
+	)
 	(bus
 		(pts
@@
 	(wire
 		(pts
-			(xy 158.75 148.59) (xy 158.75 153.67)
+			(xy 166.37 148.59) (xy 166.37 153.67)
 		)
 		(stroke
@@
 	(wire
 		(pts
-			(xy 158.75 158.75) (xy 172.72 158.75)
-		)
-		(stroke
-			(width 0)
-			(type default)
-		)
-	)
-	(wire
-		(pts
 			(xy 60.96 40.64) (xy 60.96 46.99)
 		)
@@
 	(wire
 		(pts
+			(xy 173.99 170.18) (xy 173.99 172.72)
+		)
+		(stroke
+			(width 0)
+			(type default)
+		)
+	)
+	(wire
+		(pts
 			(xy 184.15 74.93) (xy 190.5 74.93)
 		)
@@
 	(wire
 		(pts
-			(xy 187.96 161.29) (xy 195.58 161.29)
+			(xy 173.99 161.29) (xy 195.58 161.29)
 		)
 		(stroke
@@
 	(wire
 		(pts
-			(xy 158.75 148.59) (xy 172.72 148.59)
+			(xy 166.37 148.59) (xy 172.72 148.59)
 		)
 		(stroke
@@
 		)
 	)
+	(label "Ø0"
+		(at 148.59 120.65 0)
+		(effects
+			(font
+				(size 1.27 1.27)
+			)
+			(justify left bottom)
+		)
+	)
 	(label "D6"
 		(at 137.16 78.74 0)
@@
 	)
 	(global_label "~{RW}"
-		(shape input)
-		(at 226.06 139.7 0)
+		(shape output)
+		(at 215.9 140.97 0)
 		(fields_autoplaced yes)
 		(effects
@@
 		)
 		(property "Intersheetrefs" "${INTERSHEET_REFS}"
-			(at 231.7666 139.7 0)
+			(at 221.6066 140.97 0)
 			(hide yes)
 			(show_name no)
@@
 		(on_board yes)
 		(in_pos_files yes)
-		(dnp no)
+		(dnp yes)
 		(property "Reference" "C1"
 			(at 232.664 107.696 0)
@@
 		(dnp no)
 		(property "Reference" "R44"
-			(at 64.77 181.61 90)
+			(at 65.532 181.61 90)
 			(show_name no)
 			(do_not_autoplace no)
@@
 	)
 	(symbol
+		(lib_id "Device:R_Small")
+		(at 173.99 167.64 180)
+		(unit 1)
+		(body_style 1)
+		(exclude_from_sim no)
+		(in_bom yes)
+		(on_board yes)
+		(in_pos_files yes)
+		(dnp no)
+		(property "Reference" "R46"
+			(at 174.752 167.64 90)
+			(show_name no)
+			(do_not_autoplace no)
+			(effects
+				(font
+					(size 1.27 1.27)
+				)
+			)
+		)
+		(property "Value" "4k7"
+			(at 172.085 167.64 90)
+			(show_name no)
+			(do_not_autoplace no)
+			(effects
+				(font
+					(size 1.27 1.27)
+				)
+			)
+		)
+		(property "Footprint" "Resistor_THT:R_Axial_DIN0204_L3.6mm_D1.6mm_P5.08mm_Horizontal"
+			(at 173.99 167.64 0)
+			(hide yes)
+			(show_name no)
+			(do_not_autoplace no)
+			(effects
+				(font
+					(size 1.27 1.27)
+				)
+			)
+		)
+		(property "Datasheet" ""
+			(at 173.99 167.64 0)
+			(hide yes)
+			(show_name no)
+			(do_not_autoplace no)
+			(effects
+				(font
+					(size 1.27 1.27)
+				)
+			)
+		)
+		(property "Description" ""
+			(at 173.99 167.64 0)
+			(show_name no)
+			(do_not_autoplace no)
+			(effects
+				(font
+					(size 1.27 1.27)
+				)
+			)
+		)
+		(pin "1"
+		)
+		(pin "2"
+		)
+		(instances
+			(project "motherboard"
+				(path "/69b952d5-3269-40c0-8882-4a7de0153d69"
+					(reference "R46")
+					(unit 1)
+				)
+			)
+		)
+	)
+	(symbol
 		(lib_id "power:+5V")
 		(at 67.31 127 0)
@@
 	(symbol
 		(lib_id "74xx:74HC00")
-		(at 180.34 158.75 180)
+		(at 166.37 158.75 180)
 		(unit 1)
 		(body_style 1)
@@
 		(dnp no)
 		(property "Reference" "U9"
-			(at 180.34 158.75 0)
+			(at 166.37 158.75 0)
 			(show_name no)
 			(do_not_autoplace no)
@@
 		)
 		(property "Value" "74HC132"
-			(at 180.34 165.1 0)
+			(at 166.37 165.1 0)
 			(show_name no)
 			(do_not_autoplace no)
@@
 		)
 		(property "Footprint" "Package_DIP:DIP-14_W7.62mm_Socket"
-			(at 180.34 158.75 0)
+			(at 166.37 158.75 0)
 			(hide yes)
 			(show_name no)
@@
 		)
 		(property "Datasheet" "http://www.ti.com/lit/gpn/sn74hc00"
-			(at 180.34 158.75 0)
+			(at 166.37 158.75 0)
 			(hide yes)
 			(show_name no)
@@
 		)
 		(property "Description" ""
-			(at 180.34 158.75 0)
+			(at 166.37 158.75 0)
 			(show_name no)
 			(do_not_autoplace no)
@@
 	)
 	(symbol
+		(lib_id "power:GND")
+		(at 173.99 172.72 0)
+		(mirror y)
+		(unit 1)
+		(body_style 1)
+		(exclude_from_sim no)
+		(in_bom yes)
+		(on_board yes)
+		(in_pos_files yes)
+		(dnp no)
+		(property "Reference" "#PWR0127"
+			(at 173.99 179.07 0)
+			(hide yes)
+			(show_name no)
+			(do_not_autoplace no)
+			(effects
+				(font
+					(size 1.27 1.27)
+				)
+			)
+		)
+		(property "Value" "GND"
+			(at 170.434 174.498 0)
+			(show_name no)
+			(do_not_autoplace no)
+			(effects
+				(font
+					(size 1.27 1.27)
+				)
+			)
+		)
+		(property "Footprint" ""
+			(at 173.99 172.72 0)
+			(hide yes)
+			(show_name no)
+			(do_not_autoplace no)
+			(effects
+				(font
+					(size 1.27 1.27)
+				)
+			)
+		)
+		(property "Datasheet" ""
+			(at 173.99 172.72 0)
+			(hide yes)
+			(show_name no)
+			(do_not_autoplace no)
+			(effects
+				(font
+					(size 1.27 1.27)
+				)
+			)
+		)
+		(property "Description" ""
+			(at 173.99 172.72 0)
+			(show_name no)
+			(do_not_autoplace no)
+			(effects
+				(font
+					(size 1.27 1.27)
+				)
+			)
+		)
+		(pin "1"
+		)
+		(instances
+			(project "motherboard"
+				(path "/69b952d5-3269-40c0-8882-4a7de0153d69"
+					(reference "#PWR0127")
+					(unit 1)
+				)
+			)
+		)
+	)
+	(symbol
 		(lib_id "Mechanical:MountingHole")
 		(at 39.37 177.8 0)
@@
 	(symbol
 		(lib_id "74xx:74HC00")
-		(at 135.89 156.21 180)
+		(at 134.62 156.21 180)
 		(unit 2)
 		(body_style 1)
@@
 		(dnp no)
 		(property "Reference" "U9"
-			(at 135.636 156.718 0)
+			(at 134.366 156.718 0)
 			(show_name no)
 			(do_not_autoplace no)
@@
 		)
 		(property "Value" "74HC132"
-			(at 136.652 161.544 0)
+			(at 135.382 161.544 0)
 			(show_name no)
 			(do_not_autoplace no)
@@
 		)
 		(property "Footprint" "Package_DIP:DIP-14_W7.62mm_Socket"
-			(at 135.89 156.21 0)
+			(at 134.62 156.21 0)
 			(hide yes)
 			(show_name no)
@@
 		)
 		(property "Datasheet" "http://www.ti.com/lit/gpn/sn74hc00"
-			(at 135.89 156.21 0)
+			(at 134.62 156.21 0)
 			(hide yes)
 			(show_name no)
@@
 		)
 		(property "Description" ""
-			(at 135.89 156.21 0)
+			(at 134.62 156.21 0)
 			(show_name no)
 			(do_not_autoplace no)
